Commit message: edit fox description files

File: ros_packages/fox_description/urdf/base_fox_cart.gazebo.xacro (robot description, xacro)
@@ -5,8 +5,8 @@
 			<commandTopic> cmd_vel </commandTopic>
 			<odometryTopic> odom </odometryTopic>
-			<odometryFrame> map </odometryFrame>
+			<odometryFrame> odom </odometryFrame>
 			<odometrySource> world </odometrySource>
 			<publishOdomTF> true </publishOdomTF>
-			<robotBaseFrame> base_footprint </robotBaseFrame>
+			<robotBaseFrame> base_link </robotBaseFrame>
 			<publishWheelTF> false </publishWheelTF>
 			<publishTf> true </publishTf>
@@ -17,5 +17,5 @@
 			<rightJoint> wheel_right_joint </rightJoint>
 			<wheelSeparation> 0.50 </wheelSeparation>
-			<wheelDiameter> 0.1 </wheelDiameter>
+			<wheelDiameter> 0.21 </wheelDiameter>
 			<wheelAcceleration> 1 </wheelAcceleration>
 			<wheelTorque> 10 </wheelTorque>

File: ros_packages/fox_description/urdf/base_fox_cart.urdf.xacro (robot description, xacro)
@@ -18,19 +18,19 @@
 	<link name="base_link">
         <visual>
-                <origin xyz="0 0 0" rpy="0 0 0"/>
-                <geometry>
-                  <mesh	filename="package://fox_description/meshes/fox_cart.stl"
-						scale="0.001 0.001 0.001"/>
-		</geometry>
+            <origin xyz="0 0 0" rpy="0 0 0"/>
+            <geometry>
+                <mesh filename="package://fox_description/meshes/fox_cart.dae"
+					scale="0.001 0.001 0.001"/>
+			</geometry>
 		<material name="dark"/>
         </visual>
 	<collision>
-                <origin xyz="0.225 0 0.05" rpy="0 0 0"/>
-                <geometry>
-                        <box size="0.50 0.35 0.10"/>
-                </geometry>
+            <origin xyz="-0.225 0 0.05" rpy="0 0 0"/>
+            <geometry>
+                <box size="0.50 0.35 0.10"/>
+            </geometry>
 	</collision>
 	<inertial>
-                <origin xyz="0.225 0 0" rpy="0 0 0"/>
+                <origin xyz="-0.225 0 0" rpy="0 0 0"/>
                 <mass value="20"/> <!-- in kg -->
 			<!-- M=20kg, x=0.5m, y=0.34m, z=0.1m-->
@@ -39,12 +39,12 @@
         </link>
 	<!-- front_wheel macros -->
-    <xacro:front_wheel alignment="left" x_="0" y_="-0.25" z_="0" rx_="0" ry_="0" rz_="0" off_="-0.12" f_="0.01" s_="1.0"  >
+    <xacro:front_wheel alignment="left" x_="0" y_="0.25" z_="0" rx_="0" ry_="0" rz_="${pi}" off_="-0.12" f_="0.01" s_="1.0"  >
 	</xacro:front_wheel>
-    <xacro:front_wheel alignment="right" x_="0" y_="0.25" z_="0" rx_="0" ry_="0.0" rz_="${pi}" off_="0.12" f_="0.01" s_="1.0" >
+    <xacro:front_wheel alignment="right" x_="0" y_="-0.25" z_="0" rx_="0" ry_="0.0" rz_="0" off_="0.12" f_="0.01" s_="1.0" >
 	</xacro:front_wheel>
 	<!-- Caster macros -->
-    <xacro:caster alignment="left" x_="0.4" y_="-0.22" z_="-0.03" >
+    <xacro:caster alignment="left" x_="-0.4" y_="-0.22" z_="-0.03" >
 	</xacro:caster>
-    <xacro:caster alignment="right" x_="0.4" y_="0.22" z_="-0.03" >
+    <xacro:caster alignment="right" x_="-0.4" y_="0.22" z_="-0.03" >
 	</xacro:caster>
 	<!-- ar_tag macros -->

File: ros_packages/fox_description/urdf/camera.urdf.xacro (robot description, xacro)
@@ -2,5 +2,5 @@
 <robot>
   <joint name="astra_joint" type="fixed">
-    <origin xyz="-0.09 0 0.11" rpy="0 0 ${pi}"/>
+    <origin xyz="0.09 0 0.11" rpy="0 0 0"/>
     <parent link="base_link"/>
     <child link="camera_link"/>
@@ -10,5 +10,5 @@
       <origin xyz="0 0 0" rpy="${pi/2} 0 ${pi/2}"/>
       <geometry>
-        <mesh filename="package://fox_description/meshes/sensors/astra.dae" scale="0.001 0.001 0.001" />
+        <mesh filename="package://fox_description/meshes/astra.dae" scale="0.001 0.001 0.001" />
       </geometry>
     </visual>
@@ -81,5 +81,5 @@
       </plugin>
     </sensor>
-    <material>Gazebo/Grey</material>
+    <!-- <material>Gazebo/Grey</material> -->
   </gazebo>
 </robot>

File: ros_packages/fox_description/urdf/laser.urdf.xacro (robot description, xacro)
@@ -2,5 +2,5 @@
 <robot>
   <joint name="rplidar_joint" type="fixed">
-    <origin xyz="0.11 0 0.25" rpy="0 0 3.14"/>
+    <origin xyz="-0.11 0 0.25" rpy="0 0 3.14"/>
     <parent link="base_link"/>
     <child link="laser"/>
@@ -10,5 +10,5 @@
       <origin xyz="0 0 -0.15" rpy="0 0 0"/>
       <geometry>
-        <mesh filename="package://fox_description/meshes/lidar.stl" scale="0.001 0.001 0.001" />
+        <mesh filename="package://fox_description/meshes/lidar.dae" scale="0.001 0.001 0.001" />
       </geometry>
     </visual>
@@ -96,5 +96,5 @@
       </plugin>
     </sensor>
-    <material>Gazebo/Grey</material>
+    <!-- <material>Gazebo/Grey</material> -->
   </gazebo>
 </robot>

File: ros_packages/fox_description/urdf/wheel.urdf.xacro (robot description, xacro)
@@ -7,5 +7,5 @@
 			<dynamics damping="0.0005" friction="0.00" /> <!-- can be set to the right values -->
 			<!--limit upper="0.001"/--> <!-- set to correct values -->
-			<axis xyz="0 -1 0"/>
+			<axis xyz="0 1 0"/>
 			<origin xyz= "${x_} ${y_} ${z_}"/>
 		</joint>
@@ -14,5 +14,5 @@
 				<origin xyz="0 0 0" rpy="0 0 ${rz_}"/>
 				<geometry>
-					<mesh 	filename="package://fox_description/meshes/wheel_fox.stl"
+					<mesh 	filename="package://fox_description/meshes/wheel_fox.dae"
 							scale="0.001 0.001 0.001"/>
 				</geometry>
@@ -38,5 +38,5 @@
 			<mu2 value="10.0"/>
 			<fdir1>1 0 0</fdir1>
-1			<material>Gazebo/Grey</material>
+<!--			<material>Gazebo/Grey</material> -->
 		</gazebo>
 	</xacro:macro>
