Commit message: ROS2 Migration

File: fox_description/urdf/base_fox_cart.gazebo.xacro (robot description, xacro)
@@ -3,23 +3,39 @@
 	<gazebo>
 		<plugin name= "base_fox_controller" filename="libgazebo_ros_diff_drive.so" >
-			<commandTopic> cmd_vel </commandTopic>
-			<odometryTopic> odom </odometryTopic>
-			<odometryFrame> odom </odometryFrame>
-			<odometrySource> world </odometrySource>
-			<publishOdomTF> true </publishOdomTF>
-			<robotBaseFrame> base_link </robotBaseFrame>
-			<publishWheelTF> false </publishWheelTF>
-			<publishTf> true </publishTf>
-			<publishWheelJointState> true </publishWheelJointState>
-			<legacyMode> false </legacyMode>
-			<updateRate> 100 </updateRate>
-			<leftJoint> wheel_left_joint </leftJoint>
-			<rightJoint> wheel_right_joint </rightJoint>
-			<wheelSeparation> 0.50 </wheelSeparation>
-			<wheelDiameter> 0.21 </wheelDiameter>
-			<wheelAcceleration> 1 </wheelAcceleration>
-			<wheelTorque> 10 </wheelTorque>
-			<rosDebugLevel> na </rosDebugLevel>
+			<!-- <ros> -->
+                <!-- Set namespace -->
+                <!-- <namespace>/demo</namespace> -->
+                <!-- Remap default topics -->
+                <!-- <argument>cmd_vel:=cmd_demo</argument>
+                <argument>odom:=odom_demo</argument> -->
+            <!-- </ros> -->
+            <odometry_topic>odom</odometry_topic>
+            <odometry_frame> odom </odometry_frame>
+            <odometry_source> world </odometry_source>
+            <publish_odom> true </publish_odom>
+            <publish_odom_tf> true </publish_odom_tf>
+            <robot_base_frame> base_link </robot_base_frame>
+            <publish_wheel_tf> false </publish_wheel_tf>
+            <publish_tf> true </publish_tf>
+			<!-- <legacy_mode> false </legacy_mode> -->
+            <update_rate> 100 </update_rate>
+            <left_joint> wheel_left_joint </left_joint>
+            <right_joint> wheel_right_joint </right_joint>
+            <wheel_separation> 0.50 </wheel_separation>
+            <wheel_diameter> 0.21 </wheel_diameter>
+            <max_wheel_acceleration> 1 </max_wheel_acceleration>
+            <max_wheel_torque> 10 </max_wheel_torque>
+			<!-- <rosDebugLevel> na </rosDebugLevel> -->
 		</plugin>
+        <!-- Use gazebo_ros_joint_state_publisher instead of publishWheelJointState -->
+        <plugin name="joint_states" filename="libgazebo_ros_joint_state_publisher.so">
+            <ros>
+                <!-- <namespace>/fox</namespace> -->
+                <remapping>~/out:=joint_states</remapping>
+            </ros>
+            <update_rate>30</update_rate>
+            <joint_name>wheel_left_joint</joint_name>
+            <joint_name>wheel_right_joint</joint_name>
+        </plugin>
 	</gazebo>
 </robot>

File: fox_description/urdf/camera.urdf.xacro (robot description, xacro)
@@ -43,4 +43,5 @@
     <sensor type="depth" name="openni_camera_camera">
       <always_on>1</always_on>
+      <update_rate> 10.0 </update_rate>
       <visualize>true</visualize>
       <camera>
@@ -57,26 +58,40 @@
           <far>100</far>
         </clip>
+        <distortion>
+            <k1>0.0</k1>
+            <k2>0.0</k2>
+            <k3>0.0</k3>
+            <p1>0.0</p1>
+            <p2>0.0</p2>
+            <!-- <center>0.5 0.5</center> -->
+        </distortion>
       </camera>
-      <plugin name="kinect_controller" filename="libgazebo_ros_openni_kinect.so">
-        <alwaysOn>true</alwaysOn>
-        <updateRate>10.0</updateRate>
-        <cameraName>camera</cameraName>
-        <frameName>camera_depth_frame</frameName>
-        <imageTopicName>rgb/image_raw</imageTopicName>
-        <depthImageTopicName>depth/image_raw</depthImageTopicName>
-        <pointCloudTopicName>depth/points</pointCloudTopicName>
-        <cameraInfoTopicName>rgb/camera_info</cameraInfoTopicName>
-        <depthImageCameraInfoTopicName>depth/camera_info</depthImageCameraInfoTopicName>
-        <pointCloudCutoff>0.4</pointCloudCutoff>
-        <hackBaseline>0.07</hackBaseline>
-        <distortionK1>0.0</distortionK1>
-        <distortionK2>0.0</distortionK2>
-        <distortionK3>0.0</distortionK3>
-        <distortionT1>0.0</distortionT1>
-        <distortionT2>0.0</distortionT2>
+      <plugin name="kinect_controller" filename="libgazebo_ros_camera.so">
+        <always_on> true </always_on>
+        <update_rate> 10.0 </update_rate>
+        <camera_name> camera </camera_name>
+        <frame_name> camera_depth_frame </frame_name>
+        <!-- Change namespace, camera name and topics so:
+              * Raw images are published to: /custom_ns/custom_camera/custom_image
+              * Depth images are published to: /custom_ns/custom_camera/custom_image_depth
+              * Raw image camera info is published to: /custom_ns/custom_camera/custom_info_raw
+              * Depth image camera info is published to: /custom_ns/custom_camera/custom_info_depth
+              * Point cloud is published to: /custom_ns/custom_camera/custom_points
+        -->
+        <ros>
+          <!-- <namespace>custom_ns</namespace> -->
+          <argument>custom_camera/image_raw:=rgb/image_raw</argument>
+          <argument>custom_camera/image_depth:=depth/image_raw</argument>
+          <argument>custom_camera/camera_info:=rgb/camera_info</argument>
+          <argument>custom_camera/camera_info_depth:=depth/camera_info</argument>
+          <argument>custom_camera/points:=depth/points</argument>
+        </ros>
+        <!-- <pointCloudCutoff>0.4</pointCloudCutoff> -->
+        <min_depth>0.4</min_depth>
+        <hack_baseline> 0.07 </hack_baseline>
         <CxPrime>0.0</CxPrime>
         <Cx>0.0</Cx>
         <Cy>0.0</Cy>
-        <focalLength>0.0</focalLength>
+        <focal_length>0.0</focal_length>
       </plugin>
     </sensor>

File: fox_description/urdf/imu.urdf.xacro (robot description, xacro)
@@ -1,38 +1,45 @@
 <?xml version="1.0"?>
 <robot>
-  <link name="imu_link"/>
-  <joint name="imu_joint" type="fixed">
-    <parent link="base_link"/>
-    <child link="imu_link"/>
-    <origin xyz="0.0 0 0.068" rpy="0 0 0"/>
-  </joint>
-   <!-- Gazebo sensor plugin -->
-  <gazebo>
-    <plugin name= "imu_plugin" filename= "libgazebo_ros_imu.so" >
-      <always_on> true </always_on>
-      <bodyName> imu_link </bodyName>
-      <frameName> imu_link </frameName>
-      <topicName> imu </topicName>
-      <serviceName> imu_service </serviceName>
-      <gaussianNoise> 0.0 </gaussianNoise>
-      <updateRate> 200 </updateRate>
-      <imu>
-        <noise>
-          <type> gaussian </type>
-          <rate>
-            <mean> 0.0 </mean>
-            <stddev> 2e-4 </stddev>
-            <bias_mean> 0.0000075 </bias_mean>
-            <bias_stddev> 0.0000008 </bias_stddev>
-          </rate>
-          <accel>
-            <mean> 0.0 </mean>
-            <stddev> 1.7e-2 </stddev>
-            <bias_mean> 0.1 </bias_mean>
-            <bias_stddev> 0.001 </bias_stddev>
-          </accel>
-        </noise>
-      </imu>
-    </plugin>
-  </gazebo>
+    <link name="imu_link"/>
+    <joint name="imu_joint" type="fixed">
+      <parent link="base_link"/>
+      <child link="imu_link"/>
+      <origin xyz="0.0 0 0.068" rpy="0 0 0"/>
+    </joint>
+    <!-- Gazebo sensor plugin -->
+    <gazebo reference="imu_link">>
+        <sensor name="imu" type="imu">
+            <always_on>true</always_on>
+            <!-- Publish at 200 hz -->
+            <update_rate>200</update_rate>
+            <plugin name= "imu_plugin" filename= "libgazebo_ros_imu_sensor.so" >
+                <body_name> imu_link </body_name>
+                <frame_name> imu_link </frame_name>
+                <ros>
+                    <!-- Will publish to /imu/imu -->
+                    <!-- <namespace>/imu</namespace> -->
+                    <argument>~/out:=imu</argument>
+                </ros>
+                <service_name> imu_service </service_name>
+                <imu>
+                    <noise>
+                        <type> gaussian </type>
+                        <rate>
+                            <mean> 0.0 </mean>
+                            <stddev> 2e-4 </stddev>
+                            <!-- Mean and the standard deviation of the Gaussian distribution from which bias values will be sampled. -->
+                            <bias_mean> 0.0000075 </bias_mean>
+                            <bias_stddev> 0.0000008 </bias_stddev>
+                        </rate>
+                        <accel>
+                            <mean> 0.0 </mean>
+                            <stddev> 1.7e-2 </stddev>
+                            <bias_mean> 0.1 </bias_mean>
+                            <bias_stddev> 0.001 </bias_stddev>
+                        </accel>
+                    </noise>
+                </imu>
+            </plugin>
+        </sensor>
+    </gazebo>
 </robot>

File: fox_description/urdf/laser.urdf.xacro (robot description, xacro)
@@ -91,7 +91,13 @@
         </noise>
       </ray>
-      <plugin name="gazebo_ros_head_rplidar_controller" filename="libgazebo_ros_laser.so">
-        <topicName>scan</topicName>
-        <frameName>laser</frameName>
+      <plugin name="gazebo_ros_head_rplidar_controller" filename="libgazebo_ros_ray_sensor.so">
+        <frame_name> laser </frame_name>
+        <!-- Change namespace and output topic so published topic is /rrbot/laser/scan -->
+        <ros>
+            <!-- <namespace>/rrbot/laser</namespace> -->
+            <argument>~/out:=scan</argument>
+        </ros>
+        <!-- Set output to sensor_msgs/LaserScan to get same output type as gazebo_ros_laser -->
+        <output_type>sensor_msgs/LaserScan</output_type>
       </plugin>
     </sensor>
