Commit message: cleaned up extra files from legacy, added Dobots logo

File: fox_description/urdf/base_fox_cart.urdf.xacro (robot description, xacro)
@@ -3,10 +3,12 @@
 	<!--URDF uses SI Units: meters, radians and kilograms-->
 	<!-- common constants -->
-	<!--xacro:include filename="$(find fox_description)/urdf/common_properties.xacro"/-->
+	<xacro:include filename="$(find fox_description)/urdf/common_properties.xacro"/>
 	<xacro:include filename="$(find fox_description)/urdf/wheel.urdf.xacro"/>
 	<xacro:include filename="$(find fox_description)/urdf/caster.urdf.xacro"/>
 	<xacro:include filename="$(find fox_description)/urdf/camera.urdf.xacro"/>
+	<xacro:include filename="$(find fox_description)/urdf/imu.urdf.xacro"/>
 	<xacro:include filename="$(find fox_description)/urdf/laser.urdf.xacro"/>
-<!--	<xacro:include filename="$(find fox_description)/urdf/ar_tag.urdf.xacro"/> -->
+	<xacro:include filename="$(find fox_description)/urdf/logo.urdf.xacro"/>
+	<!-- <xacro:include filename="$(find fox_description)/urdf/ar_tag.urdf.xacro"/> -->
 	<!-- Base
 	<link name="base_footprint"/>
@@ -23,19 +25,19 @@
 					scale="0.001 0.001 0.001"/>
 			</geometry>
-		<material name="dark"/>
+			<material name="dark"/>
         </visual>
-	<collision>
-            <origin xyz="-0.225 0 0.05" rpy="0 0 0"/>
-            <geometry>
-                <box size="0.50 0.35 0.10"/>
-            </geometry>
-	</collision>
-	<inertial>
-                <origin xyz="-0.225 0 0" rpy="0 0 0"/>
-                <mass value="20"/> <!-- in kg -->
+		<collision>
+			<origin xyz="-0.225 0 0.05" rpy="0 0 0"/>
+			<geometry>
+				<box size="0.50 0.35 0.10"/>
+			</geometry>
+		</collision>
+		<inertial>
+			<origin xyz="-0.225 0 0" rpy="0 0 0"/>
+			<mass value="20"/> <!-- in kg -->
 			<!-- M=20kg, x=0.5m, y=0.34m, z=0.1m-->
-                <inertia ixx="0.2093333" ixy="0.0" ixz="0.0" iyy="0.4333333" iyz="0.0" izz="0.6093333"/>
+			<inertia ixx="0.2093333" ixy="0.0" ixz="0.0" iyy="0.4333333" iyz="0.0" izz="0.6093333"/>
         </inertial>
-        </link>
+	</link>
 	<!-- front_wheel macros -->
     <xacro:front_wheel alignment="left" x_="0" y_="0.25" z_="0" rx_="0" ry_="0" rz_="${pi}" off_="-0.12" f_="0.01" s_="1.0"  >
@@ -48,6 +50,9 @@
     <xacro:caster alignment="right" x_="-0.4" y_="0.22" z_="-0.03" >
 	</xacro:caster>
+	<!-- logo macro -->
+	<xacro:logo_tag x_="-0.28" y_="0.0" z_="0.0975" r_="0" p_="0" yaw_="0">
+	</xacro:logo_tag>
 	<!-- ar_tag macros -->
-<!--    <xacro:ar_tag number_="5" x_="0.0" y_="0.0" z_="0.15" r_="0.0">
+	<!-- <xacro:ar_tag number_="5" x_="0.0" y_="0.0" z_="0.15" r_="0.0">
 	</xacro:ar_tag> -->
 	<!-- Gazebo simulation plugins -->

File: fox_description/urdf/laser.urdf.xacro (robot description, xacro)
@@ -14,5 +14,5 @@
     </visual>
     <collision>
-      <origin xyz="0 0 0.04" rpy="0 0 0"/>
+      <origin xyz="0 0 -0.1" rpy="0 0 0"/>
       <geometry>
         <box size="0.08 0.08 0.08"/>

File: fox_description/urdf/logo.urdf.xacro (robot description, xacro)
@@ -1,34 +1,34 @@
 <?xml version="1.0"?>
-<robot xmlns:xacro="http://ros.org/wiki/xacro" name="ar_tag">
-	<xacro:macro name="ar_tag" params="number_ x_ y_ z_ r_">
-		<link name="ar_tag_${number_}">
+<robot xmlns:xacro="http://ros.org/wiki/xacro" name="logo_tag">
+	<xacro:macro name="logo_tag" params="x_ y_ z_ r_ p_ yaw_">
+		<link name="logo_tag">
 			<visual>
+				<origin xyz="0 0 0" rpy="0 0 0"/>
+				<geometry>
+					<box size="0.28 0.175 0.0001"/>
+				</geometry>
+			</visual>
+			<!-- <inertial>
+				<origin xyz="0 0 0"/>
+				<mass value="0.001" />
+				<inertia ixx="0.000001" ixy="0.0" ixz="0.0" iyy= "0.000001" iyz="0.0" izz="0.000001" />
+			</inertial> -->
+			<!-- <collision>
 				<origin xyz="0 0 0" rpy="0 0 0"/>
 				<geometry>
 					<box size="0.5 0.5 0.03"/>
 				</geometry>
-			</visual>
-			<inertial>
-				<origin xyz="0 0 0"/>
-				<mass value="0.001" />
-				<inertia ixx="0.000001" ixy="0.0" ixz="0.0" iyy= "0.000001" iyz="0.0" izz="0.000001" />
-			</inertial>
-			<collision>
-				<origin xyz="0 0 0" rpy="0 0 0"/>
-				<geometry>
-					<box size="0.5 0.5 0.03"/>
-				</geometry>
-			</collision>
+			</collision> -->
 		</link>
-		<joint name="ar_tag_${number_}_joint" type="fixed">
+		<joint name="logo_tag_joint" type="fixed">
 			<parent link="base_link"/>
-			<child link="ar_tag_${number_}"/>
-			<origin xyz= "${x_} ${y_} ${z_}" rpy="0.0 ${r_} 0.0"/>
+			<child link="logo_tag"/>
+			<origin xyz= "${x_} ${y_} ${z_}" rpy="${r_} ${p_} ${yaw_}"/>
 		</joint>
-		<gazebo reference="ar_tag_${number_}">
+		<gazebo reference="logo_tag">
 			<kp value="50000000.0" />
 			<kd value="0.2" />
 			<minDepth>0.001</minDepth>
-			<material>ar_tag_13 </material>
+			<material>logo</material>
 		</gazebo>
 	</xacro:macro>

Commit message: xacro fixes for spawn

File: fox_description/urdf/base_fox_cart.urdf.xacro (robot description, xacro)
@@ -11,11 +11,11 @@
 	<xacro:include filename="$(find fox_description)/urdf/logo.urdf.xacro"/>
 	<!-- <xacro:include filename="$(find fox_description)/urdf/ar_tag.urdf.xacro"/> -->
-	<!-- Base
-	<link name="base_footprint"/>
-	<joint name="base_joint" type="fixed">
-		<origin xyz="0 0 0.105" rpy="0 0 0"/>
-                <parent link="base_footprint"/>
-	        <child link="base_link"/>
-	</joint> -->
+	<!-- Base -->
+	<!-- <link name="base_footprint"/> -->
+	<!-- <joint name="base_joint" type="fixed"> -->
+		<!-- <origin xyz="0 0 0.105" rpy="0 0 0"/> -->
+                <!-- <parent link="base_footprint"/> -->
+	        <!-- <child link="base_link"/> -->
+	<!-- </joint> -->
 	<link name="base_link">
         <visual>
@@ -54,6 +54,5 @@
 	</xacro:logo_tag>
 	<!-- ar_tag macros -->
-	<!-- <xacro:ar_tag number_="5" x_="0.0" y_="0.0" z_="0.15" r_="0.0">
-	</xacro:ar_tag> -->
+	<!-- <xacro:ar_tag number_="5" x_="0.0" y_="0.0" z_="0.15" r_="0.0"/>-->
 	<!-- Gazebo simulation plugins -->
 	<xacro:include filename="$(find fox_description)/urdf/base_fox_cart.gazebo.xacro"/>

File: fox_description/urdf/base_fox_cart_verticaltag.urdf.xacro (robot description, xacro)
@@ -70,6 +70,5 @@
 	</xacro:caster>
 	<!-- ar_tag macros -->
-    <xacro:ar_tag number_="5" x_="-0.3" y_="0.0" z_="0.35" r_="1.0" >
-	</xacro:ar_tag>
+    <xacro:ar_tag number_="5" x_="-0.3" y_="0.0" z_="0.35" r_="1.0" />
 	<!-- Gazebo simulation plugins -->
 	<xacro:include filename="$(find fox_description)/urdf/base_fox_cart.gazebo.xacro"/>

File: fox_description/urdf/caster.urdf.xacro (robot description, xacro)
@@ -10,11 +10,10 @@
 		</joint>
 		<link name="caster_${alignment}_link">
-<!--			<visual>
-				<origin xyz="0 0 0" rpy="${pi/2} 0 0"/>
-				<geometry>
-					<cylinder length="0.01" radius="0.057"/>
-				</geometry>
-			</visual>
--->
+			<!-- <visual> -->
+				<!-- <origin xyz="0 0 0" rpy="${pi/2} 0 0"/> -->
+				<!-- <geometry> -->
+					<!-- <cylinder length="0.01" radius="0.057"/> -->
+				<!-- </geometry> -->
+			<!-- </visual> -->
 			<inertial>
 				<origin xyz="0 0 0"/>

File: fox_description/urdf/logo.urdf.xacro (robot description, xacro)
@@ -9,15 +9,15 @@
 				</geometry>
 			</visual>
-			<!-- <inertial>
-				<origin xyz="0 0 0"/>
-				<mass value="0.001" />
-				<inertia ixx="0.000001" ixy="0.0" ixz="0.0" iyy= "0.000001" iyz="0.0" izz="0.000001" />
-			</inertial> -->
-			<!-- <collision>
-				<origin xyz="0 0 0" rpy="0 0 0"/>
-				<geometry>
-					<box size="0.5 0.5 0.03"/>
-				</geometry>
-			</collision> -->
+			<!-- <inertial> -->
+				<!-- <origin xyz="0 0 0"/> -->
+				<!-- <mass value="0.001" /> -->
+				<!-- <inertia ixx="0.000001" ixy="0.0" ixz="0.0" iyy= "0.000001" iyz="0.0" izz="0.000001" /> -->
+			<!-- </inertial> -->
+			<!-- <collision> -->
+				<!-- <origin xyz="0 0 0" rpy="0 0 0"/> -->
+				<!-- <geometry> -->
+					<!-- <box size="0.5 0.5 0.03"/> -->
+				<!-- </geometry> -->
+			<!-- </collision> -->
 		</link>
 		<joint name="logo_tag_joint" type="fixed">

File: fox_description/urdf/wheel.urdf.xacro (robot description, xacro)
@@ -38,5 +38,5 @@
 			<mu2 value="10.0"/>
 			<fdir1>1 0 0</fdir1>
-<!--			<material>Gazebo/Grey</material> -->
+			<!-- <material>Gazebo/Grey</material> -->
 		</gazebo>
 	</xacro:macro>
